File: hardware/PCB/Liquorice_PCB/TB6612FNG.kicad_sch (KiCad schematic)
At the start: 5 parts, among them U2 TB6612FNG

Commit message: Added BOM and finialized main schematic.
Parts:
- added J3, J4: Conn_01x02_Pin, Connector_PinHeader_2.54mm:PinHeader_1x02_P2.54mm_Vertical, symbol Connector:Conn_01x02_Pin
Connections:
- net VCC is gone; now on net +3.3V: C1.1, C3.2, U2.20 (VCC)
- net AO1: no longer names the net of U2.1 (AO1), U2.2 (AO1)
- net AO1: now also J3.2 (Pin_2)
- net AO2: no longer names the net of U2.5 (AO2), U2.6 (AO2)
- net AO2: now also J3.1 (Pin_1)
- net BO1: no longer names the net of U2.11 (BO1), U2.12 (BO1)
- net BO1: now also J4.2 (Pin_2)
- net BO2: no longer names the net of U2.7 (BO2), U2.8 (BO2)
- net BO2: now also J4.1 (Pin_1)
- net STBY renamed +3.3V
