File: hardware/PCB/Liquorice_PCB/Liquorice_PCB.kicad_sch (KiCad schematic)
At the start: 2 parts, among them J1 Conn_01x19_Pin, J2 Conn_01x19_Pin

Commit message: Added BOM and finialized main schematic.
Parts:
- added C10, C5, C6, C7: 100nF, Capacitor_SMD:C_0805_2012Metric_Pad1.18x1.45mm_HandSolder, symbol Device:C
- added C8, C9: 10uF, Capacitor_Tantalum_SMD:CP_EIA-3216-18_Kemet-A_HandSolder, symbol Device:C_Polarized_Small
- added J3, J4, J5, J6, J7: Conn_01x02_Pin, Connector_PinHeader_2.54mm:PinHeader_1x02_P2.54mm_Vertical, symbol Connector:Conn_01x02_Pin
- added U1: TB6612FNG, Package_SO:SSOP-24_5.3x8.2mm_P0.65mm, symbol Driver_Motor:TB6612FNG
- added U3: BMI320, Package_LGA:Bosch_LGA-14_3x2.5mm_P0.5mm, symbol New_Library:BMI320
Connections:
- net CS: now also J1.7 (Pin_7), U3.12 (CSB); no longer J1.4 (Pin_4)
- net MISO: now also J2.11 (Pin_11), U3.1 (SDO); no longer J2.12 (Pin_12)
- net MOSI: now also J2.10 (Pin_10), U3.14 (SDx); no longer J2.11 (Pin_11)
- net SCK: now also J2.9 (Pin_9), U3.13 (SCx); no longer J2.10 (Pin_10)
- net +3.3V: now reaches J2.1 (Pin_1)
- net +3.3V: now also C5.1, C6.1, C7.2, C8.1, U1.19 (STBY), U1.20 (VCC), U3.5 (VDDIO), U3.8 (VDD)
- net AIN1: now reaches J2.13 (Pin_13)
- net AIN1: now also U1.21 (AIN1)
- net GND: now reaches J2.14 (Pin_14)
- net GND: now also J1.13 (Pin_13), J1.19 (Pin_19), C10.2, C5.2, C6.2, C7.1, C8.2, C9.2, J3.1 (Pin_1), U1.10 (PGND2), U1.18 (GND), U1.3 (PGND1), U1.4 (PGND1), U1.9 (PGND2), U3.6 (GNDIO), U3.7 (GND)
- net BIN1: now reaches J2.15 (Pin_15)
- net BIN1: now also U1.17 (BIN1)
- net +5V: now reaches J2.19 (Pin_19)
- net +5V: now also C10.1, C9.1, J3.2 (Pin_2), U1.13 (VM2), U1.14 (VM3), U1.24 (VM1)
- net PWMB: now reaches J2.7 (Pin_7)
- net PWMB: now also U1.15 (PWMB)
- net BIN2: now reaches J2.8 (Pin_8)
- net BIN2: now also U1.16 (BIN2)
- net at J1.11 (Pin_11): now also J4.1 (Pin_1)
- net at J1.12 (Pin_12): now also J4.2 (Pin_2)
- net at J1.17 (Pin_17): now also J7.1 (Pin_1)
- net at J1.18 (Pin_18): now also J7.2 (Pin_2)
- new net: J5.1 (Pin_1), U1.5 (AO2), U1.6 (AO2)
- new net: J5.2 (Pin_2), U1.1 (AO1), U1.2 (AO1)
- new net: J6.2 (Pin_2), U1.11 (BO1), U1.12 (BO1)
- new net: J6.1 (Pin_1), U1.7 (BO2), U1.8 (BO2)
- new net AIN2: J1.4 (Pin_4), U1.22 (AIN2)
- new net PWMA: J2.12 (Pin_12), U1.23 (PWMA)
- no-connect marks 0 -> 21
Other:
- removed sheet IMU
- removed sheet Motor_Driver
- note added: "BMI320 IMU"
- note added: "Battery connection"
- note added: "Encoder 1 SDA on top pin"
- note added: "Encoder 2 SDA on top pin"
- note added: "Motor driver"
- note added: "Super accurate ESP32 symbol"
- moved on the sheet: J1, J2

Commit message: Finalized PCB schematic and layout
Parts:
- added R1, R2, R3, R4: 5.1k, Resistor_SMD:R_0603_1608Metric_Pad0.98x0.95mm_HandSolder, symbol Device:R
- renumbered J3 to J1, J7 to J2, J4 to J3, J5 to J4, J6 to J5, J1 to J6, J2 to J7
Connections:
- net +3.3V: now also R1.1, R2.1, R3.1, R4.1
- net at J3.1 (Pin_1), J6.11 (Pin_11): now also R4.2
- net at J3.2 (Pin_2), J6.12 (Pin_12): now also R3.2
- net at J2.1 (Pin_1), J6.17 (Pin_17): now also R2.2
- net at J2.2 (Pin_2), J6.18 (Pin_18): now also R1.2
